File: OptoTap/Tap_Photosensor_PCB_v2/Tap_Photosensor_PCB.kicad_sch (KiCad schematic)
At the start: 10 parts, among them J1 Conn_01x03, U1 OPB961N51, U2 AP63205WU

Commit message: updated kicad files with proper resistor values
Parts:
- R1: value R200 -> 200R
- R3: value R640 -> 640R
Changed lines of the file:
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@@
       (effects (font (size 1.27 1.27)) (justify left))
     )
-    (property "Value" "R200" (id 1) (at 105.918 76.7966 0)
+    (property "Value" "200R" (id 1) (at 105.918 76.7966 0)
       (effects (font (size 1.27 1.27)) (justify left))
     )
@@
       (effects (font (size 1.27 1.27)) (justify left))
     )
-    (property "Value" "R640" (id 1) (at 179.578 60.2866 0)
+    (property "Value" "640R" (id 1) (at 179.578 60.2866 0)
       (effects (font (size 1.27 1.27)) (justify left))
     )
@@
     )
     (path "/42af5c76-1be1-40a2-9d2a-448b0eb158cf"
-      (reference "R1") (unit 1) (value "R200") (footprint "Resistor_SMD:R_0603_1608Metric")
+      (reference "R1") (unit 1) (value "200R") (footprint "Resistor_SMD:R_0603_1608Metric")
     )
     (path "/dbb9bcbf-c2e0-477c-8d37-a9e225856a7d"
-      (reference "R3") (unit 1) (value "R640") (footprint "Resistor_SMD:R_0603_1608Metric")
+      (reference "R3") (unit 1) (value "640R") (footprint "Resistor_SMD:R_0603_1608Metric")
     )
     (path "/a3d4a3b8-80b2-4158-b88b-eda5110f79c7"

Commit message: updated OptoTap boards
Parts:
- removed D1: LED, LED_SMD:LED_0603_1608Metric, symbol Device:LED
- added C4: 68 nF, Capacitor_SMD:C_0402_1005Metric, symbol Device:C_Small
- added C5: 22 µF, Capacitor_SMD:C_0603_1608Metric, symbol Device:C_Small
- added D1: XL-1615RGBC, LED_SMD:LED_0606_1432, symbol LED:XL-1615RBGC
- added D3: D_Schottky, Diode_SMD:D_SOD-323, symbol Device:D_Schottky
- added F1: Polyfuse_Small, Resistor_SMD:R_0805_2012Metric, symbol Device:Polyfuse_Small
- added JP1: SolderJumper_3_Bridged12, Jumper:SolderJumper-3_P1.3mm_Bridged12_RoundedPad1.0x1.5mm_NumberLabels, symbol Jumper:SolderJumper_3_Bridged12
- added JP2: SolderJumper_2_Bridged, Jumper:SolderJumper-2_DARKMODE, symbol Jumper:SolderJumper_2_Bridged
- C1: LCSC (none) -> C440198; PARTNUM (none) -> GRM21BR61H106KE43L
- C2: value 220 nF -> 100 nF; footprint Capacitor_SMD:C_0805_2012Metric -> Capacitor_SMD:C_0402_1005Metric; LCSC (none) -> C307331; PARTNUM (none) -> CL05B104KB54PNC
- C3: footprint Capacitor_SMD:C_0805_2012Metric -> Capacitor_SMD:C_0603_1608Metric; LCSC (none) -> C84419; PARTNUM (none) -> GRM188R61A226ME15D
- L1: footprint Inductor_SMD:L_0805_2012Metric -> Inductor_SMD:CKCS3010; LCSC (none) -> C354557; PARTNUM (none) -> CKCS3012-4.7uH/M
- R1: LCSC (none) -> C8218; PARTNUM (none) -> 0603WAF2000T5E
- R3: value 640R -> 620R; LCSC (none) -> C23220; PARTNUM (none) -> 0603WAF6200T5E
- U1: footprint OPTO_OPB961N51 -> footprints:OPTO_EE-SX398_OPB666N
- U2: LCSC (none) -> C2071056; PARTNUM (none) -> AP63205WU
Connections:
- net +5V: now also JP1.2 (C), JP2.2 (B); no longer C3.1, L1.2, R3.1, U2.1 (FB)
- net GND: now also C4.2, C5.2, D1.3 (B)
- net SIG: now also D1.1 (R)
- net Vin: now also D3.2 (A); no longer C1.1, U2.2 (EN), U2.3 (IN)
- net at R3.2: now also D1.2 (A)
- net sw_node: now reaches C2.1, L1.1, U2.5 (SW)
- net bst: now reaches C2.2, U2.6 (BST)
- new net: C4.1, U2.2 (EN)
- new net: JP2.1 (A), R3.1
- new net Vcc: D3.1 (K), F1.1, JP1.3 (B)
- new net fb: C3.1, C5.1, JP1.1 (A), L1.2, U2.1 (FB)
- new net fuse_out: C1.1, F1.2, U2.3 (IN)
- no-connect marks 0 -> 1
Other:
- moved on the sheet: C1, C2, C3, J1, L1, R1, R3, U1, U2

Commit message: Opto24 (#68)
* updated OptoTap boards

* updated inductor info

* updated STEP and kicad

* updated README with LED ordering info

* fixed bad save
Connections:
- net LED+: now reaches D1.2 (A), R3.2
Changed lines of the file:
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@@
-    (stroke (width 0) (type default))
-  )
-  (wire (pts (xy 127 73.66) (xy 127 81.28))
     (stroke (width 0) (type default))
   )
@@
   )
   (wire (pts (xy 191.77 78.74) (xy 191.77 97.79))
+    (stroke (width 0) (type default))
+  )
+  (wire (pts (xy 127 73.66) (xy 127 81.28))
     (stroke (width 0) (type default))
   )
@@
     (stroke (width 0) (type default))
   )
+  (label "B" (at 132.08 77.47 0) (fields_autoplaced)
+    (effects (font (size 1.27 1.27)) (justify left bottom))
+  )
   (label "bst" (at 214.63 76.2 0) (fields_autoplaced)
     (effects (font (size 1.27 1.27)) (justify left bottom))
   )
   (label "fuse_out" (at 165.1 59.69 0) (fields_autoplaced)
+    (effects (font (size 1.27 1.27)) (justify left bottom))
+  )
+  (label "LED+" (at 132.08 63.5 0) (fields_autoplaced)
     (effects (font (size 1.27 1.27)) (justify left bottom))
   )
@@
     (effects (font (size 1.27 1.27)) (justify left bottom))
   )
+  (label "R" (at 127 77.47 0) (fields_autoplaced)
+    (effects (font (size 1.27 1.27)) (justify left bottom))
+  )
